File: _autosave-Digitiyer_demo_1V8_module.kicad_sch (KiCad schematic)
At the start: 56 parts, among them J1 Conn_01x08, J2 Conn_01x24, J3 Conn_01x04_Pin, J4 USB_C_Receptacle_PowerOnly_6P, Q2 SI1308EDL, U2 LM27762DSSR, U3 TMUX1108PWR, U4 RF-BM-ND05, U5 TPS63900DSKR, U6 TXB0108PWR, U8 74LVC1G34GW

Commit message: aktualizace
Parts:
- added D7: LESD5Z5_0T1G, Diode_SMD:D_SOD-523, symbol JLCImport:LESD5Z5_0T1G
Connections:
- net at C35.2, U5.1 (EN), U5.10 (VIN)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: now also D7.1 (C); no longer J4.A9 (VBUS), J4.B9 (VBUS)
- new net: D7.2 (A), J4.A9 (VBUS), J4.B9 (VBUS)
Changed lines of the file:
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@@
 	(wire
 		(pts
-			(xy 44.45 34.29) (xy 57.15 34.29)
+			(xy 44.45 34.29) (xy 45.72 34.29)
+		)
+		(stroke
+			(width 0)
+			(type default)
+		)
+	)
+	(wire
+		(pts
+			(xy 55.88 34.29) (xy 57.15 34.29)
 		)
 		(stroke
@@
 					(unit 1)
 				)
+			)
+		)
+	)
+	(symbol
+		(lib_id "JLCImport:LESD5Z5_0T1G")
+		(at 50.8 34.29 180)
+		(unit 1)
+		(exclude_from_sim no)
+		(in_bom yes)
+		(on_board yes)
+		(dnp no)
+		(fields_autoplaced yes)
+		(property "Reference" "D7"
+			(at 51.054 26.67 0)
+			(effects
+				(font
+					(size 1.27 1.27)
+				)
+			)
+		)
+		(property "Value" "LESD5Z5_0T1G"
+			(at 51.054 29.21 0)
+			(effects
+				(font
+					(size 1.27 1.27)
+				)
+			)
+		)
+		(property "Footprint" "Diode_SMD:D_SOD-523"
+			(at 50.8 34.29 0)
+			(effects
+				(font
+					(size 1.27 1.27)
+				)
+				(hide yes)
+			)
+		)
+		(property "Datasheet" "https://www.lcsc.com/datasheet/lcsc_datasheet_1811021122_LRC-LESD5Z5-0T1G_C136171.pdf"
+			(at 50.8 34.29 0)
+			(effects
+				(font
+					(size 1.27 1.27)
+				)
+				(hide yes)
+			)
+		)
+		(property "Description" "-40℃~+125℃ 174W@8/20us 18.6V 1uA 5V 6.2V 80pF 9.4A@8/20us IEC 61000-4-2、IEC 61000-4-4 TVS Unidirectional SOD-523 ESD and Surge Protection (TVS/ESD) ROHS"
+			(at 50.8 34.29 0)
+			(effects
+				(font
+					(size 1.27 1.27)
+				)
+				(hide yes)
+			)
+		)
+		(property "LCSC" "C136171"
+			(at 50.8 34.29 0)
+			(effects
+				(font
+					(size 1.27 1.27)
+				)
+				(hide yes)
+			)
+		)
+		(property "Manufacturer" "LRC"
+			(at 50.8 34.29 0)
+			(effects
+				(font
+					(size 1.27 1.27)
+				)
+				(hide yes)
+			)
+		)
+		(property "Manufacturer Part" "LESD5Z5.0T1G"
+			(at 50.8 34.29 0)
+			(effects
+				(font
+					(size 1.27 1.27)
+				)
+				(hide yes)
+			)
+		)
+		(pin "1"
+		)
+		(pin "2"
+		)
+		(instances
+			(project ""
+				(path "/9366839b-90ab-4146-a727-74c5e521354c"
+					(reference "D7")
+					(unit 1)
+				)
