File: Digitiyer_demo_1V8_module.kicad_pcb (KiCad board)
At the start: 2 copper layers, 35 x 35 mm, 93 parts, among them J1 Conn_01x08, J2 Conn_01x24, Q1 AO3400A, Q2 SI1308EDL, U1 Opamp_Quad, U2 LM27762DSSR, U3 TMUX1108PWR, U4 RF-BM-ND05, U5 TPS63900DSKR, U6 TXB0108PWR, U8 74LVC1G34GW

Commit message: aktualizace
Parts:
- added D7: LESD5Z5_0T1G, Diode_SMD:D_SOD-523, F.Cu at (181.2, 92.9)
- added J3: Conn_01x04_Pin, Connector_PinHeader_2.54mm:PinHeader_1x04_P2.54mm_Vertical, F.Cu at (166.4, 79.6)
- added J4: USB_C_Receptacle_PowerOnly_6P, Connector_USB:USB_C_Receptacle_HRO_TYPE-C-31-M-17, F.Cu at (184.2, 98.1)
- added R27: 5.1k, Capacitor_SMD:C_0402_1005Metric, F.Cu at (183.5, 92.8)
- added R9: 5.1k, Capacitor_SMD:C_0402_1005Metric, F.Cu at (185.3, 92.7)
- added REF**: TestPoint_Pad_D1.0mm, TestPoint:TestPoint_Pad_D1.0mm, B.Cu at (158.4, 69.0)
- added REF**: TestPoint_Pad_D1.0mm, TestPoint:TestPoint_Pad_D1.0mm, B.Cu at (155.8, 69.0)
- J2, NT1: moved to B.Cu
- moved L1 113.3 mm to (186.8, 68.3), turned to 90 degrees
- moved C28 111.3 mm to (187.8, 89.3), turned to 180 degrees
- moved C26 111.2 mm to (187.8, 84.7), turned to 180 degrees
- moved C27 111.1 mm to (187.8, 87.8), turned to 180 degrees
- moved C25 110.4 mm to (187.8, 86.2), turned to 180 degrees
- moved C32 109.7 mm to (185.4, 71.5)
- moved C31 109.5 mm to (187.8, 76.5), turned to -90 degrees
- moved Q2 106.1 mm to (177.9, 77.2)
- moved C24 105.7 mm to (182.4, 80.8)
- moved C30 105.5 mm to (187.8, 92.3), turned to 180 degrees
- moved C29 105.3 mm to (187.8, 90.8), turned to 180 degrees
- moved D6 103.3 mm to (188.1, 72.7), turned to 90 degrees
- moved C33 102.2 mm to (180.1, 81.2), turned to -90 degrees
- moved R21 99.0 mm to (182.4, 79.2)
- moved D4 98.6 mm to (188.1, 81.6), turned to 90 degrees
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Connections:
- C23 pad 1: /AFE/INTG -> INTG
- D3 pad 1: /AFE/INTG -> INTG
- J2 pad 1: /NC -> unconnected-(J2-Pin_1-Pad1)
- J2 pad 4: /NC -> unconnected-(J2-Pin_4-Pad4)
- R29 pad 1: /AFE/INTG -> INTG
- U4 pad 13: /AIN0 -> INTG
- U4 pad 28: unconnected-(U4-SWDIO-Pad28) -> /SWDIO
- U4 pad 29: unconnected-(U4-SWCLK-Pad29) -> /SWCLK
- U6 pad 1: /SDI_1V8 -> /BUSY_1V8
- U6 pad 14: /BUSY -> /RES
- U6 pad 15: /RES -> /D/C
- U6 pad 16: /D/C -> /CS
- U6 pad 17: /CS -> /SDI
- U6 pad 20: /SDI -> /BUSY
- U6 pad 4: /CS_1V8 -> /SDI_1V8
- U6 pad 5: /D/C_1V8 -> /CS_1V8
- U6 pad 6: /RES_1V8 -> /D/C_1V8
- U6 pad 7: /BUSY_1V8 -> /RES_1V8
Routing:
- net GND: track 22.2 -> 98.3 mm, vias 7 -> 30
- net +1V8: track 3.84 -> 57.7 mm, vias 0 -> 6
- net VSSA: track 21.4 -> 74.2 mm, vias 17 -> 18
- net VDD: track 4.94 -> 49.6 mm, vias 0 -> 5
- net +3V3: track 1.72 -> 39.9 mm, vias 0 -> 5
- net VEE: track 1.45 -> 38.8 mm, vias 0 -> 2
- net DISCHARGE: track 0.00 -> 33.7 mm, vias 0 -> 2
- net /RES_1V8: track 0.00 -> 32.7 mm, vias 0 -> 2
- net /A0: track 0.00 -> 31.9 mm, vias 0 -> 2
- net INTG: track 0.00 -> 31.3 mm, vias 0 -> 2
- net VDDA: track 2.25 -> 32.5 mm, vias 0 -> 2
- net /D/C_1V8: track 0.00 -> 28.7 mm, vias 0 -> 2
- net /A1: track 0.00 -> 27.5 mm, vias 0 -> 2
- net Net-(D6-A): track 0.00 -> 26.9 mm
- net /CS_1V8: track 0.00 -> 25.2 mm, vias 0 -> 2
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- added copper zone on B.Cu, net GND
- added copper zone on F.Cu, net GND
- removed copper zone on F.Cu, net +3V3
Other:
- board size 35 x 35 mm -> 37.8 x 35 mm
- board text added: "1V8"
- board text added: "2026"
- board text added: "AFE"
- board text added: "GND"
- board text added: "Prototyp 1: test EMR+EPD Robin Josef Šafařík, 2026"
- board text added: "SWCLK"
- board text added: "SWDIO"
- board text added: "VSSA"

Commit message: uložení
Parts:
- added REF**: TestPoint_Pad_D1.0mm, TestPoint:TestPoint_Pad_D1.0mm, B.Cu at (175.4, 84.2)
- added REF**: TestPoint_Pad_D1.0mm, TestPoint:TestPoint_Pad_D1.0mm, B.Cu at (179.9, 75.1)
- added REF**: TestPoint_Pad_D1.0mm, TestPoint:TestPoint_Pad_D1.0mm, B.Cu at (155.7, 77.4)
- added REF**: TestPoint_Pad_D1.0mm, TestPoint:TestPoint_Pad_D1.0mm, B.Cu at (156.1, 99.1)
Connections:
- C35 pad 2: Net-(D7-C) -> Net-(D7-A)
- D7 pad 1: Net-(D7-C) -> GND
- U3 pad 2: /EN -> VDDA
- U5 pad 1: Net-(D7-C) -> Net-(D7-A)
- U5 pad 10: Net-(D7-C) -> Net-(D7-A)
- U5 pad 2: Net-(D7-C) -> Net-(D7-A)
Routing:
- net Net-(D7-A): track 10.6 -> 39.7 mm, vias 0 -> 2
- net Net-(D7-C): track 28.5 -> 0.00 mm, vias 2 -> 0
- net VDDA: track 32.5 -> 38.0 mm, vias 2 -> 3
- net VEE: track 38.8 -> 42.0 mm
- net GND: track 98.3 -> 101.0 mm
- net +3V3: track 39.9 -> 41.7 mm
- net +1V8: track 57.7 -> 59.1 mm
Other:
- board text added: "3V3"
- board text added: "Trim"
- board text added: "VDDA"
- board text added: "VEE"
- board text removed: "Prototyp 1: test EMR+EPD Robin Josef Šafařík, 2026"

Commit message: uložit
Parts:
- C36, C37: value 0.1uF -> 100nF
- J2: footprint JLCImport:05B20U24P -> JLCImport:FPC-0_5FX-24PWBH15
- U7: value ~ -> 74LVC1G34GW
- moved REF** 0.60 mm to (179.9, 74.5)
- moved D6 0.45 mm to (188.1, 73.2)
- moved C31 0.45 mm to (187.8, 77.0)
- moved C32 0.20 mm to (185.4, 71.7)
- moved C35 0.20 mm to (184.5, 76.7)
- moved L1 0.20 mm to (186.8, 68.5)
- moved R23 0.18 mm to (184.7, 74.1)
Routing:
- net GND: track 101.0 -> 107.0 mm, vias 30 -> 33
- net VSSA: track 74.2 -> 75.5 mm, vias 18 -> 19
- net Net-(D6-A): track 26.9 -> 28.1 mm

Commit message: uložit
Parts:
- moved D7 0.11 mm to (181.3, 92.8)
- moved R27 0.05 mm to (183.5, 92.8)
Connections:
- C35 pad 2: Net-(D7-A) -> Net-(D7-C)
- D7 pad 1: GND -> Net-(D7-C)
- D7 pad 2: Net-(D7-A) -> GND
- J4 pad A9: Net-(D7-A) -> Net-(D7-C)
- J4 pad B9: Net-(D7-A) -> Net-(D7-C)
- U5 pad 1: Net-(D7-A) -> Net-(D7-C)
- U5 pad 10: Net-(D7-A) -> Net-(D7-C)
- U5 pad 2: Net-(D7-A) -> Net-(D7-C)
Routing:
- net Net-(D7-A): track 39.4 -> 0.00 mm, vias 2 -> 0
- net Net-(D7-C): track 0.00 -> 38.3 mm, vias 0 -> 2
- net GND: track 107.0 -> 108.6 mm

Commit message: nové uložení
Parts:
- removed R5: 10k, Resistor_SMD:R_0805_2012Metric
- moved REF** 1.10 mm to (180.8, 75.2)
- moved C1 0.71 mm to (177.8, 67.3)
- moved C5 0.56 mm to (180.3, 67.0)
- moved C37 0.56 mm to (184.4, 68.2)
- moved R4 0.19 mm to (183.3, 70.9)
- moved C32 0.15 mm to (185.6, 71.7)
- moved R2 0.09 mm to (178.1, 69.3)
- moved D6 0.08 mm to (188.2, 73.2)
- moved C3 0.07 mm to (181.5, 71.3)
- moved R1 0.06 mm to (176.6, 69.3)
- moved R3 0.05 mm to (183.2, 67.8)
Connections:
- U2 pad 1: Net-(U2-PGOOD) -> GND
- U2 pad 12: unconnected-(U2-EN+-Pad12) -> +3V3
- U2 pad 8: unconnected-(U2-EN–-Pad8) -> +3V3
Routing:
- net GND: track 108.6 -> 129.5 mm, vias 33 -> 32
- net +3V3: track 41.4 -> 48.8 mm, vias 5 -> 9
- net Net-(U2-PGOOD): track 1.93 -> 0.00 mm
- net VDD: track 49.6 -> 47.9 mm
- net Net-(U2-FB+): track 4.70 -> 5.45 mm

Commit message: uložitt
Parts:
- removed R24: 50k, Resistor_SMD:R_0603_1608Metric
- Q2: footprint Package_TO_SOT_SMD:SOT-23-3 -> Package_TO_SOT_SMD:SOT-323_SC-70_Handsoldering
- U7: value 74LVC1G34GW -> OPA365AQDBVRQ1
- moved Q2 0.61 mm to (178.3, 77.7)
- moved REF** 0.05 mm to (156.0, 99.1)
Connections:
- U6 pad 10: Net-(U6-OE) -> +1V8
- U7 pad 1: /AFE/OP3O -> Net-(R13-Pad2)
- U7 pad 2: Net-(U7--) -> /AFE/OPAMP_-
- U7 pad 3: /AFE/OPAMP_+ -> /AFE/OP3O
- U7 pad 4: /AFE/OPAMP_- -> Net-(U7--)
- U7 pad 5: Net-(R13-Pad2) -> /AFE/OPAMP_+
Routing:
- net +1V8: track 59.1 -> 73.9 mm, vias 6 -> 7
- net Net-(U6-OE): track 13.3 -> 0.00 mm
- net VSSA: track 75.5 -> 87.8 mm
- net /AFE/OP3O: track 9.48 -> 12.7 mm
- net /AFE/OPAMP_-: track 25.9 -> 29.0 mm, vias 3 -> 4
- net GND: track 129.5 -> 127.0 mm
- net Net-(U7--): track 11.3 -> 12.9 mm, vias 1 -> 2
- net Net-(D6-A): track 27.9 -> 26.6 mm
- net +3V3: track 48.8 -> 49.9 mm
- net Net-(D2-A): track 7.49 -> 8.41 mm
- net Net-(D7-C): track 38.3 -> 37.6 mm
- net Net-(R13-Pad2): track 13.0 -> 12.5 mm
- net /AFE/OPAMP_+: track 28.6 -> 28.0 mm
- net VEE: track 42.0 -> 42.5 mm

Commit message: uklad
Parts:
- added C39: 10uF, Capacitor_SMD:C_0402_1005Metric, F.Cu at (178.4, 82.2)
- added C40: 100nF, Capacitor_SMD:C_0603_1608Metric, F.Cu at (163.8, 79.6)
- added REF**: TestPoint_Pad_D1.0mm, TestPoint:TestPoint_Pad_D1.0mm, B.Cu at (187.6, 73.8)
- added REF**: TestPoint_Pad_D1.0mm, TestPoint:TestPoint_Pad_D1.0mm, B.Cu at (175.3, 87.7)
- added REF**: TestPoint_Pad_D1.0mm, TestPoint:TestPoint_Pad_D1.0mm, B.Cu at (155.7, 83.6)
- added REF**: TestPoint_Pad_D1.0mm, TestPoint:TestPoint_Pad_D1.0mm, B.Cu at (186.4, 95.2)
- R10, R11, R12, R15, R17, R18, R27, R29, R6, R9: footprint Capacitor_SMD:C_0402_1005Metric -> Resistor_SMD:R_0402_1005Metric
- R14, R16, R19, R25, R26, R7, R8: footprint Capacitor_SMD:C_0805_2012Metric -> Resistor_SMD:R_0805_2012Metric
- R20: footprint Capacitor_SMD:C_0603_1608Metric -> Resistor_SMD:R_0603_1608Metric
Routing:
- net GND: track 127.0 -> 140.2 mm
- net +1V8: track 73.9 -> 83.0 mm, vias 7 -> 8
- net /PREVGL: track 15.8 -> 24.1 mm
- net /SWCLK: track 18.7 -> 21.3 mm
- net /SWDIO: track 16.6 -> 18.5 mm
- net INTG: track 31.3 -> 32.9 mm
- net /PREVGH: track 20.5 -> 21.5 mm, vias 1 -> 2
- net /VCOM: track 7.35 -> 6.51 mm
Other:
- board text added: "INTG"

Commit message: finální uložení?
Parts:
- added D8: LED_Small, LED_SMD:LED_0603_1608Metric, F.Cu at (162.4, 79.6)
- FB1, FB2, FB3, FB4, FB5: footprint Capacitor_SMD:C_0805_2012Metric -> Inductor_SMD:L_0805_2012Metric
- U1: value Opamp_Quad -> COS8054TR
- moved C36 0.13 mm to (173.3, 73.6)
- moved FB5 0.06 mm to (159.1, 99.2)
Connections:
- U1 pad 10: /AFE/OP3M -> VSSA
- U1 pad 12: /AFE/OP4M -> VSSA
- U1 pad 13: VSSA -> /AFE/OP4M
- U1 pad 2: VSSA -> /AFE/OP1M
- U1 pad 3: /AFE/OP1M -> VSSA
- U1 pad 5: /AFE/OP2M -> VSSA
- U1 pad 6: VSSA -> /AFE/OP2M
- U1 pad 9: VSSA -> /AFE/OP3M
- U4 pad 14: unconnected-(U4-P03-Pad14) -> Net-(D8-A)
Routing:
- net Net-(D8-A): track 0.00 -> 12.9 mm
- net /SWDIO: track 18.5 -> 23.7 mm
- net GND: track 140.2 -> 143.5 mm
- net /SWCLK: track 21.3 -> 23.3 mm
- net VSSA: track 87.6 -> 88.2 mm
- net /AFE/OP4M: track 6.27 -> 6.80 mm
- net /AFE/OP1M: track 4.07 -> 4.58 mm
