File: Digitiyer_demo_1V8_module.kicad_pcb (KiCad board)
At the start: 2 copper layers, 37.8 x 35 mm, 109 parts, among them J1 Conn_01x08, J2 Conn_01x24, J3 Conn_01x04_Pin, J4 USB_C_Receptacle_PowerOnly_6P, Q1 AO3400A, Q2 SI1308EDL, U1 COS8054TR, U2 LM27762DSSR, U3 TMUX1108PWR, U4 RF-BM-ND05, U5 TPS63900DSKR, U6 TXB0108PWR, U7 OPA365AQDBVRQ1, U8 74LVC1G34GW

Commit message: save
Parts:
- C31, C33: footprint Capacitor_SMD:C_0603_1608Metric -> Capacitor_SMD:C_0805_2012Metric
- moved C31 0.24 mm to (187.8, 77.2)
- moved C25 0.15 mm to (187.8, 86.4)
- moved C33 0.15 mm to (179.9, 81.2)
- moved C27 0.11 mm to (187.8, 87.9)
- moved D4 0.10 mm to (188.1, 81.7)
- moved C26 0.08 mm to (187.8, 84.8)
- moved C28 0.06 mm to (187.8, 89.3)
Routing:
- net VDD: track 47.9 -> 48.7 mm
- net +3V3: track 49.9 -> 50.6 mm
- net /PREVGH: track 21.4 -> 22.1 mm
- net /GDR: track 14.1 -> 14.7 mm
