File: analog.kicad_sch (KiCad schematic)
At the start: 39 parts, among them Q1 AO3400A, U1 Opamp_Quad, U7 ${SIM.PARAMS}

Commit message: uložit
Parts:
- U7: value ${SIM.PARAMS} -> 74LVC1G34GW
Changed lines of the file:
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@@
 		(on_board yes)
 		(dnp no)
-		(fields_autoplaced yes)
 		(property "Reference" "U7"
-			(at 129.54 110.4198 0)
+			(at 122.428 108.458 0)
 			(effects
 				(font
@@
 			)
 		)
-		(property "Value" "${SIM.PARAMS}"
-			(at 129.54 112.3249 0)
+		(property "Value" "74LVC1G34GW"
+			(at 128.016 111.0549 0)
 			(effects
 				(font

Commit message: uložitt
Parts:
- U7: value 74LVC1G34GW -> OPA365AQDBVRQ1
Connections:
- net OP3O: now also U7.3 (+); no longer U7.1 (+)
- net OPAMP_+: now also U7.5 (V+); no longer U7.3 (V+)
- net OPAMP_-: now also U7.2 (V-); no longer U7.4 (V-)
- net at R13.2, R15.2: now also U7.1; no longer U7.5
- net at R10.1, R11.2: now also U7.4 (-); no longer U7.2 (-)
Other:
- note added: "PPD"
Changed lines of the file:
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@@
 	(generator_version "9.0")
 	(paper "A4")
+	(text "PPD"
+		(exclude_from_sim no)
+		(at 125.73 120.65 0)
+		(effects
+			(font
+				(size 1.27 1.27)
+			)
+		)
+	)
 	(text "High-pass min 60 kHz"
 		(exclude_from_sim no)
@@
 		)
 	)
+	(text "PPD"
+		(exclude_from_sim no)
+		(at 120.904 70.866 0)
+		(effects
+			(font
+				(size 1.27 1.27)
+			)
+		)
+	)
+	(text "PPD"
+		(exclude_from_sim no)
+		(at 184.15 87.122 0)
+		(effects
+			(font
+				(size 1.27 1.27)
+			)
+		)
+	)
 	(junction
 		(at 101.6 55.88)
@@
 			)
 		)
-		(property "Value" "74LVC1G34GW"
-			(at 128.016 111.0549 0)
+		(property "Value" "OPA365AQDBVRQ1"
+			(at 130.048 110.998 0)
 			(effects
 				(font
@@
 		)
 		(property "Sim.Library" "${KICAD9_SYMBOL_DIR}/Simulation_SPICE.sp"
-			(at 121.92 115.57 0)
+			(at 122.174 115.316 0)
 			(effects
 				(font

Commit message: uklad
Parts:
- R10, R11, R12, R15, R17, R18, R29, R6: footprint Capacitor_SMD:C_0402_1005Metric -> Resistor_SMD:R_0402_1005Metric
- R14, R16, R19, R25, R26, R7, R8: footprint Capacitor_SMD:C_0805_2012Metric -> Resistor_SMD:R_0805_2012Metric
Changed lines of the file:
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@@
 			)
 		)
-		(property "Footprint" "Capacitor_SMD:C_0805_2012Metric"
+		(property "Footprint" "Resistor_SMD:R_0805_2012Metric"
 			(at 189.23 67.31 0)
 			(effects
@@
 			)
 		)
-		(property "Footprint" "Capacitor_SMD:C_0805_2012Metric"
+		(property "Footprint" "Resistor_SMD:R_0805_2012Metric"
 			(at 90.17 67.31 0)
 			(effects
@@
 			)
 		)
-		(property "Footprint" "Capacitor_SMD:C_0402_1005Metric"
+		(property "Footprint" "Resistor_SMD:R_0402_1005Metric"
 			(at 130.81 59.69 0)
 			(effects
@@
 			)
 		)
-		(property "Footprint" "Capacitor_SMD:C_0805_2012Metric"
+		(property "Footprint" "Resistor_SMD:R_0805_2012Metric"
 			(at 101.6 59.69 0)
 			(effects
@@
 			)
 		)
-		(property "Footprint" "Capacitor_SMD:C_0805_2012Metric"
+		(property "Footprint" "Resistor_SMD:R_0805_2012Metric"
 			(at 201.93 59.69 0)
 			(effects
@@
 			)
 		)
-		(property "Footprint" "Capacitor_SMD:C_0402_1005Metric"
+		(property "Footprint" "Resistor_SMD:R_0402_1005Metric"
 			(at 111.76 124.46 0)
 			(effects
@@
 			)
 		)
-		(property "Footprint" "Capacitor_SMD:C_0402_1005Metric"
+		(property "Footprint" "Resistor_SMD:R_0402_1005Metric"
 			(at 205.74 109.22 0)
 			(effects
@@
 			)
 		)
-		(property "Footprint" "Capacitor_SMD:C_0805_2012Metric"
+		(property "Footprint" "Resistor_SMD:R_0805_2012Metric"
 			(at 135.89 67.31 0)
 			(effects
@@
 			)
 		)
-		(property "Footprint" "Capacitor_SMD:C_0402_1005Metric"
+		(property "Footprint" "Resistor_SMD:R_0402_1005Metric"
 			(at 170.18 106.68 0)
 			(effects
@@
 			)
 		)
-		(property "Footprint" "Capacitor_SMD:C_0805_2012Metric"
+		(property "Footprint" "Resistor_SMD:R_0805_2012Metric"
 			(at 148.59 59.69 0)
 			(effects
@@
 			)
 		)
-		(property "Footprint" "Capacitor_SMD:C_0402_1005Metric"
+		(property "Footprint" "Resistor_SMD:R_0402_1005Metric"
 			(at 69.85 59.69 0)
 			(effects
@@
 			)
 		)
-		(property "Footprint" "Capacitor_SMD:C_0402_1005Metric"
+		(property "Footprint" "Resistor_SMD:R_0402_1005Metric"
 			(at 175.26 59.69 0)
 			(effects
@@
 			)
 		)
-		(property "Footprint" "Capacitor_SMD:C_0402_1005Metric"
+		(property "Footprint" "Resistor_SMD:R_0402_1005Metric"
 			(at 125.73 102.87 0)
 			(effects
@@
 			)
 		)
-		(property "Footprint" "Capacitor_SMD:C_0805_2012Metric"
+		(property "Footprint" "Resistor_SMD:R_0805_2012Metric"
 			(at 175.26 85.09 0)
 			(effects
@@
 			)
 		)
-		(property "Footprint" "Capacitor_SMD:C_0402_1005Metric"
+		(property "Footprint" "Resistor_SMD:R_0402_1005Metric"
 			(at 146.05 106.68 0)
 			(effects

Commit message: finální uložení?
Parts:
- FB4, FB5: footprint Capacitor_SMD:C_0805_2012Metric -> Inductor_SMD:L_0805_2012Metric
- U1: value Opamp_Quad -> COS8054TR
Connections:
- net OP1M: now also U1.2 (-); no longer U1.3 (+)
- net OP2M: now also U1.6 (-); no longer U1.5 (+)
- net OP3M: now also U1.9 (-); no longer U1.10 (+)
- net OP4M: now also U1.13 (-); no longer U1.12 (+)
- net VSSA: now also U1.10 (+), U1.12 (+), U1.3 (+), U1.5 (+); no longer U1.13 (-), U1.2 (-), U1.6 (-), U1.9 (-)
Other:
- moved on the sheet: R18
Changed lines of the file:
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@@
 	)
 	(junction
+		(at 218.44 147.32)
+		(diameter 0)
+		(color 0 0 0 0)
+	)
+	(junction
 		(at 101.6 55.88)
 		(diameter 0)
@@
 	)
 	(junction
+		(at 218.44 132.08)
+		(diameter 0)
+		(color 0 0 0 0)
+	)
+	(junction
 		(at 148.59 63.5)
 		(diameter 0)
@@
 	(wire
 		(pts
-			(xy 177.8 59.69) (xy 189.23 59.69)
+			(xy 181.61 59.69) (xy 189.23 59.69)
 		)
 		(stroke
@@
 	(wire
 		(pts
-			(xy 104.14 68.58) (xy 104.14 83.82)
+			(xy 104.14 68.58) (xy 104.14 69.85)
 		)
 		(stroke
@@
 	(wire
 		(pts
-			(xy 172.72 59.69) (xy 170.18 59.69)
+			(xy 176.53 59.69) (xy 170.18 59.69)
 		)
 		(stroke
@@
 		(dnp no)
 		(property "Reference" "U1"
-			(at 191.262 104.648 0)
+			(at 191.516 104.648 0)
 			(effects
 				(font
@@
 			)
 		)
-		(property "Value" "Opamp_Quad"
+		(property "Value" "COS8054TR"
 			(at 190.5 101.6 0)
 			(effects
@@
 	)
 	(symbol
+		(lib_name "Opamp_Quad_3")
 		(lib_id "Device:Opamp_Quad")
 		(at 162.56 66.04 0)
@@
 		(dnp no)
 		(property "Reference" "U1"
-			(at 164.084 61.468 0)
+			(at 163.576 61.468 0)
 			(effects
 				(font
@@
 			)
 		)
-		(property "Value" "Opamp_Quad"
+		(property "Value" "COS8054TR"
 			(at 162.56 58.42 0)
 			(effects
@@
 	)
 	(symbol
+		(lib_name "Opamp_Quad_2")
 		(lib_id "Device:Opamp_Quad")
 		(at 215.9 66.04 0)
@@
 		(dnp no)
 		(property "Reference" "U1"
-			(at 216.916 61.214 0)
+			(at 216.916 61.468 0)
 			(effects
 				(font
@@
 			)
 		)
-		(property "Value" "Opamp_Quad"
+		(property "Value" "COS8054TR"
 			(at 215.9 58.42 0)
 			(effects
@@
 			)
 		)
-		(property "Footprint" "Capacitor_SMD:C_0805_2012Metric"
+		(property "Footprint" "Inductor_SMD:L_0805_2012Metric"
 			(at 198.628 129.54 90)
 			(effects
@@
 	)
 	(symbol
+		(lib_name "Opamp_Quad_1")
 		(lib_id "Device:Opamp_Quad")
 		(at 199.39 139.7 0)
@@
 		(on_board yes)
 		(dnp no)
-		(fields_autoplaced yes)
 		(property "Reference" "U1"
-			(at 198.12 139.6999 0)
+			(at 200.406 135.128 0)
 			(effects
 				(font
 					(size 1.27 1.27)
 				)
-				(justify left)
 			)
 		)
-		(property "Value" "Opamp_Quad"
-			(at 198.12 140.9699 0)
+		(property "Value" "COS8054TR"
+			(at 186.944 139.192 0)
 			(effects
 				(font
 					(size 1.27 1.27)
 				)
-				(justify left)
-				(hide yes)
 			)
 		)
@@
 	)
 	(symbol
+		(lib_id "power:PWR_FLAG")
+		(at 218.44 147.32 180)
+		(unit 1)
+		(exclude_from_sim no)
+		(in_bom yes)
+		(on_board yes)
+		(dnp no)
+		(fields_autoplaced yes)
+		(property "Reference" "#FLG010"
+			(at 218.44 149.225 0)
+			(effects
+				(font
+					(size 1.27 1.27)
+				)
+				(hide yes)
+			)
+		)
+		(property "Value" "PWR_FLAG"
+			(at 218.44 152.4 0)
+			(effects
+				(font
+					(size 1.27 1.27)
+				)
+				(hide yes)
+			)
+		)
+		(property "Footprint" ""
+			(at 218.44 147.32 0)
+			(effects
+				(font
+					(size 1.27 1.27)
+				)
+				(hide yes)
+			)
+		)
+		(property "Datasheet" "~"
+			(at 218.44 147.32 0)
+			(effects
+				(font
+					(size 1.27 1.27)
+				)
+				(hide yes)
+			)
+		)
+		(property "Description" "Special symbol for telling ERC where power comes from"
+			(at 218.44 147.32 0)
+			(effects
+				(font
+					(size 1.27 1.27)
+				)
+				(hide yes)
+			)
+		)
+		(pin "1"
+		)
+		(instances
+			(project "Digitiyer_demo_1V8_module"
+				(path "/9366839b-90ab-4146-a727-74c5e521354c/da421d0b-f626-4bbe-a076-4662d67f0e17"
+					(reference "#FLG010")
+					(unit 1)
+				)
+			)
+		)
+	)
+	(symbol
 		(lib_id "Device:FerriteBead_Small")
 		(at 196.85 149.86 180)
@@
 			)
 		)
-		(property "Footprint" "Capacitor_SMD:C_0805_2012Metric"
+		(property "Footprint" "Inductor_SMD:L_0805_2012Metric"
 			(at 198.628 149.86 90)
 			(effects
@@
 	)
 	(symbol
+		(lib_name "Opamp_Quad_4")
 		(lib_id "Device:Opamp_Quad")
 		(at 118.11 66.04 0)
@@
 			)
 		)
-		(property "Value" "Opamp_Quad"
+		(property "Value" "COS8054TR"
 			(at 118.11 58.42 0)
 			(effects
@@
 	(symbol
 		(lib_id "Device:R_Small")
-		(at 175.26 59.69 270)
+		(at 179.07 59.69 270)
 		(unit 1)
 		(exclude_from_sim no)
@@
 		(dnp no)
 		(property "Reference" "R18"
-			(at 174.625 55.245 90)
+			(at 178.435 55.245 90)
 			(effects
 				(font
@@
 		)
 		(property "Value" "470"
-			(at 175.133 57.531 90)
+			(at 178.943 57.531 90)
 			(effects
 				(font
@@
 		)
 		(property "Footprint" "Resistor_SMD:R_0402_1005Metric"
-			(at 175.26 59.69 0)
+			(at 179.07 59.69 0)
 			(effects
 				(font
@@
 		)
 		(property "Datasheet" "~"
-			(at 175.26 59.69 0)
+			(at 179.07 59.69 0)
 			(effects
 				(font
@@
 		)
 		(property "Description" "Resistor, small symbol"
-			(at 175.26 59.69 0)
+			(at 179.07 59.69 0)
 			(effects
 				(font
@@
 		(dnp no)
 		(property "Reference" "R19"
-			(at 175.006 83.058 90)
+			(at 175.26 83.058 90)
 			(effects
 				(font
@@
 		)
 		(property "Value" "10K"
-			(at 175.26 86.868 90)
+			(at 175.26 87.376 90)
 			(effects
 				(font
@@
 	(symbol
 		(lib_id "power:VSSA")
-		(at 104.14 83.82 180)
+		(at 104.14 69.85 180)
 		(unit 1)
 		(exclude_from_sim no)
@@
 		(fields_autoplaced yes)
 		(property "Reference" "#PWR021"
-			(at 104.14 80.01 0)
+			(at 104.14 66.04 0)
 			(effects
 				(font
@@
 		)
 		(property "Value" "VSSA"
-			(at 104.14 88.9 0)
+			(at 104.14 74.93 0)
 			(effects
 				(font
@@
 		)
 		(property "Footprint" ""
-			(at 104.14 83.82 0)
+			(at 104.14 69.85 0)
 			(effects
 				(font
@@
 		)
 		(property "Datasheet" ""
-			(at 104.14 83.82 0)
+			(at 104.14 69.85 0)
 			(effects
 				(font
@@
 		)
 		(property "Description" "Power symbol creates a global label with name \"VSSA\""
-			(at 104.14 83.82 0)
+			(at 104.14 69.85 0)
 			(effects
 				(font
@@
 					(unit 1)
 				)
+			)
+		)
+	)
+	(symbol
+		(lib_id "power:PWR_FLAG")
+		(at 218.44 132.08 0)
+		(unit 1)
+		(exclude_from_sim no)
+		(in_bom yes)
+		(on_board yes)
+		(dnp no)
+		(fields_autoplaced yes)
+		(property "Reference" "#FLG09"
+			(at 218.44 130.175 0)
+			(effects
+				(font
+					(size 1.27 1.27)
+				)
+				(hide yes)
+			)
+		)
+		(property "Value" "PWR_FLAG"
+			(at 218.44 127 0)
+			(effects
+				(font
+					(size 1.27 1.27)
+				)
+				(hide yes)
+			)
+		)
+		(property "Footprint" ""
+			(at 218.44 132.08 0)
+			(effects
+				(font
+					(size 1.27 1.27)
+				)
+				(hide yes)
+			)
+		)
+		(property "Datasheet" "~"
+			(at 218.44 132.08 0)
+			(effects
+				(font
+					(size 1.27 1.27)
+				)
+				(hide yes)
+			)
+		)
+		(property "Description" "Special symbol for telling ERC where power comes from"
+			(at 218.44 132.08 0)
+			(effects
+				(font
+					(size 1.27 1.27)
+				)
+				(hide yes)
+			)
+		)
+		(pin "1"
+		)
+		(instances
+			(project "Digitiyer_demo_1V8_module"
+				(path "/9366839b-90ab-4146-a727-74c5e521354c/da421d0b-f626-4bbe-a076-4662d67f0e17"
+					(reference "#FLG09")
+					(unit 1)
+				)
