File: Digitiyer_demo_1V8_module.kicad_sch (KiCad schematic)
At the start: 56 parts, among them J1 Conn_01x08, J2 Conn_01x24, J3 Conn_01x04_Pin, J4 USB_C_Receptacle_PowerOnly_6P, Q2 SI1308EDL, U2 LM27762DSSR, U3 TMUX1108PWR, U4 RF-BM-ND05, U5 TPS63900DSKR, U6 TXB0108PWR, U8 74LVC1G34GW

Commit message: uložení
Parts:
- added D7: LESD5Z5_0T1G, Diode_SMD:D_SOD-523, symbol JLCImport:LESD5Z5_0T1G
Connections:
- net EN is gone; now on net VDDA: U3.2 (EN)
- net GND: now also D7.1 (C)
- net at C35.2, J4.A9 (VBUS), J4.B9 (VBUS)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: now also D7.2 (A)
- no-connect marks 13 -> 32

Commit message: uložit
Parts:
- C36, C37: value 0.1uF -> 100nF
- J2: footprint JLCImport:05B20U24P -> JLCImport:FPC-0_5FX-24PWBH15
Changed lines of the file:
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@@
 			)
 		)
-		(property "Value" "0.1uF"
+		(property "Value" "100nF"
 			(at 266.446 38.1 0)
 			(effects
@@
 			)
 		)
-		(property "Value" "0.1uF"
+		(property "Value" "100nF"
 			(at 206.756 38.354 0)
 			(effects
@@
 			)
 		)
-		(property "Footprint" "JLCImport:05B20U24P"
+		(property "Footprint" "JLCImport:FPC-0_5FX-24PWBH15"
 			(at 271.78 104.14 0)
 			(effects

Commit message: uložit
Connections:
- net GND: now also D7.2 (A); no longer D7.1 (C)
- net at C35.2, J4.A9 (VBUS), J4.B9 (VBUS)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: now also D7.1 (C); no longer D7.2 (A)
Other:
- note added: "Zkontrolováno."
- moved on the sheet: D7
Changed lines of the file:
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@@
 		)
 	)
+	(text "Zkontrolováno."
+		(exclude_from_sim no)
+		(at 106.68 193.294 0)
+		(effects
+			(font
+				(size 1.27 1.27)
+			)
+		)
+	)
 	(text "VHG"
 		(exclude_from_sim no)
@@
 		)
 	)
+	(text "Zkontrolováno."
+		(exclude_from_sim no)
+		(at 273.812 138.43 0)
+		(effects
+			(font
+				(size 1.27 1.27)
+			)
+		)
+	)
 	(junction
 		(at 77.47 148.59)
@@
 	)
 	(junction
+		(at 48.26 34.29)
+		(diameter 0)
+		(color 0 0 0 0)
+	)
+	(junction
 		(at 199.39 132.08)
 		(diameter 0)
@@
 	)
 	(junction
-		(at 48.26 34.29)
-		(diameter 0)
-		(color 0 0 0 0)
-	)
-	(junction
 		(at 57.15 34.29)
 		(diameter 0)
@@
 	)
 	(junction
+		(at 57.15 44.45)
+		(diameter 0)
+		(color 0 0 0 0)
+	)
+	(junction
 		(at 179.07 105.41)
 		(diameter 0)
@@
 	)
 	(junction
-		(at 57.15 44.45)
-		(diameter 0)
-		(color 0 0 0 0)
-	)
-	(junction
 		(at 223.52 105.41)
 		(diameter 0)
@@
 	(wire
 		(pts
+			(xy 57.15 44.45) (xy 57.15 45.72)
+		)
+		(stroke
+			(width 0)
+			(type default)
+		)
+	)
+	(wire
+		(pts
 			(xy 139.7 128.27) (xy 139.7 133.35)
 		)
@@
 	(wire
 		(pts
-			(xy 48.26 34.29) (xy 57.15 34.29)
-		)
-		(stroke
-			(width 0)
-			(type default)
-		)
-	)
-	(wire
-		(pts
 			(xy 204.47 92.71) (xy 210.82 92.71)
 		)
@@
 	(wire
 		(pts
-			(xy 57.15 41.91) (xy 57.15 44.45)
-		)
-		(stroke
-			(width 0)
-			(type default)
-		)
-	)
-	(wire
-		(pts
 			(xy 254 86.36) (xy 266.7 86.36)
 		)
@@
 	(wire
 		(pts
+			(xy 57.15 41.91) (xy 57.15 44.45)
+		)
+		(stroke
+			(width 0)
+			(type default)
+		)
+	)
+	(wire
+		(pts
 			(xy 173.99 153.67) (xy 181.61 153.67)
 		)
@@
 	(wire
 		(pts
+			(xy 48.26 34.29) (xy 57.15 34.29)
+		)
+		(stroke
+			(width 0)
+			(type default)
+		)
+	)
+	(wire
+		(pts
 			(xy 218.44 92.71) (xy 220.98 92.71)
 		)
@@
 	(wire
 		(pts
-			(xy 57.15 44.45) (xy 57.15 45.72)
-		)
-		(stroke
-			(width 0)
-			(type default)
-		)
-	)
-	(wire
-		(pts
 			(xy 81.28 185.42) (xy 81.28 187.96)
 		)
@@
 	(symbol
 		(lib_id "JLCImport:LESD5Z5_0T1G")
-		(at 48.26 39.37 90)
+		(at 48.26 39.37 270)
 		(unit 1)
 		(exclude_from_sim no)
@@
 		(dnp no)
 		(property "Reference" "D7"
-			(at 45.466 29.21 90)
+			(at 51.054 49.53 90)
 			(effects
 				(font
@@
 		)
 		(property "Value" "LESD5Z5_0T1G"
-			(at 45.466 31.75 90)
+			(at 51.054 46.99 90)
 			(effects
 				(font

Commit message: nové uložení
Parts:
- removed R5: 10k, Resistor_SMD:R_0805_2012Metric, symbol Device:R_Small
Connections:
- net +3V3: now also U2.12 (EN+), U2.8 (EN–)
- net GND: now also U2.1 (PGOOD)
- no-connect marks 32 -> 30
Other:
- note added: "SPD"

Commit message: uložitt
Parts:
- removed R24: 50k, Resistor_SMD:R_0603_1608Metric, symbol Device:R_Small
- Q2: footprint Package_TO_SOT_SMD:SOT-23-3 -> Package_TO_SOT_SMD:SOT-323_SC-70_Handsoldering
Connections:
- net +1V8: now also U6.10 (OE)
Changed lines of the file:
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@@
 		)
 	)
+	(text "SPD"
+		(exclude_from_sim no)
+		(at 86.36 181.356 0)
+		(effects
+			(font
+				(size 1.27 1.27)
+			)
+		)
+	)
 	(text "Součástky ANO"
 		(exclude_from_sim no)
@@
 		)
 	)
+	(text "SPD"
+		(exclude_from_sim no)
+		(at 33.02 163.83 0)
+		(effects
+			(font
+				(size 1.27 1.27)
+			)
+		)
+	)
 	(text "Součástky ANO"
 		(exclude_from_sim no)
@@
 		)
 	)
+	(text "SPD"
+		(exclude_from_sim no)
+		(at 225.044 62.484 0)
+		(effects
+			(font
+				(size 1.27 1.27)
+			)
+		)
+	)
 	(text "Use low-ESR ceramic multi-layer capacitors"
 		(exclude_from_sim no)
@@
 		)
 	)
+	(text "SPD"
+		(exclude_from_sim no)
+		(at 56.388 113.538 0)
+		(effects
+			(font
+				(size 1.27 1.27)
+			)
+		)
+	)
 	(text "Zkontrolováno."
 		(exclude_from_sim no)
@@
 	(wire
 		(pts
-			(xy 220.98 58.42) (xy 220.98 57.15)
-		)
-		(stroke
-			(width 0)
-			(type default)
-		)
-	)
-	(wire
-		(pts
 			(xy 76.2 24.13) (xy 76.2 27.94)
 		)
@@
 	(wire
 		(pts
-			(xy 220.98 64.77) (xy 220.98 63.5)
-		)
-		(stroke
-			(width 0)
-			(type default)
-		)
-	)
-	(wire
-		(pts
 			(xy 27.94 85.09) (xy 27.94 86.36)
 		)
@@
 	(wire
 		(pts
-			(xy 220.98 57.15) (xy 227.33 57.15)
-		)
-		(stroke
-			(width 0)
-			(type default)
-		)
-	)
-	(wire
-		(pts
 			(xy 245.11 129.54) (xy 242.57 129.54)
 		)
@@
 	(wire
 		(pts
+			(xy 214.63 57.15) (xy 227.33 57.15)
+		)
+		(stroke
+			(width 0)
+			(type default)
+		)
+	)
+	(wire
+		(pts
 			(xy 118.11 97.79) (xy 125.73 97.79)
 		)
@@
 	)
 	(symbol
-		(lib_id "power:GND")
-		(at 220.98 64.77 0)
-		(unit 1)
-		(exclude_from_sim no)
-		(in_bom yes)
-		(on_board yes)
-		(dnp no)
-		(property "Reference" "#PWR036"
-			(at 220.98 71.12 0)
-			(effects
-				(font
-					(size 1.27 1.27)
-				)
-				(hide yes)
-			)
-		)
-		(property "Value" "GND"
-			(at 221.107 69.1642 0)
-			(effects
-				(font
-					(size 1.27 1.27)
-				)
-			)
-		)
-		(property "Footprint" ""
-			(at 220.98 64.77 0)
-			(effects
-				(font
-					(size 1.27 1.27)
-				)
-				(hide yes)
-			)
-		)
-		(property "Datasheet" ""
-			(at 220.98 64.77 0)
-			(effects
-				(font
-					(size 1.27 1.27)
-				)
-				(hide yes)
-			)
-		)
-		(property "Description" "Power symbol creates a global label with name \"GND\" , ground"
-			(at 220.98 64.77 0)
-			(effects
-				(font
-					(size 1.27 1.27)
-				)
-				(hide yes)
-			)
-		)
-		(pin "1"
-		)
-		(instances
-			(project "Digitiyer_demo_1V8_module"
-				(path "/9366839b-90ab-4146-a727-74c5e521354c"
-					(reference "#PWR036")
-					(unit 1)
-				)
-			)
-		)
-	)
-	(symbol
 		(lib_id "Device:R_Small")
 		(at 76.2 93.98 180)
@@
 	)
 	(symbol
-		(lib_id "Device:R_Small")
-		(at 220.98 60.96 180)
-		(unit 1)
-		(exclude_from_sim no)
-		(in_bom yes)
-		(on_board yes)
-		(dnp no)
-		(property "Reference" "R24"
-			(at 223.52 60.198 0)
-			(effects
-				(font
-					(size 1.016 1.016)
-				)
-			)
-		)
-		(property "Value" "50k"
-			(at 224.028 62.23 0)
-			(effects
-				(font
-					(size 1.27 1.27)
-				)
-			)
-		)
-		(property "Footprint" "Resistor_SMD:R_0603_1608Metric"
-			(at 220.98 60.96 0)
-			(effects
-				(font
-					(size 1.27 1.27)
-				)
-				(hide yes)
-			)
-		)
-		(property "Datasheet" "~"
-			(at 220.98 60.96 0)
-			(effects
-				(font
-					(size 1.27 1.27)
-				)
-				(hide yes)
-			)
-		)
-		(property "Description" "Resistor, small symbol"
-			(at 220.98 60.96 0)
-			(effects
-				(font
-					(size 1.27 1.27)
-				)
-				(hide yes)
-			)
-		)
-		(pin "1"
-		)
-		(pin "2"
-		)
-		(instances
-			(project "Digitiyer_demo_1V8_module"
-				(path "/9366839b-90ab-4146-a727-74c5e521354c"
-					(reference "R24")
-					(unit 1)
-				)
-			)
-		)
-	)
-	(symbol
 		(lib_id "power:+3V3")
 		(at 264.16 31.75 0)
@@
 	)
 	(symbol
+		(lib_id "power:+1V8")
+		(at 214.63 57.15 0)
+		(unit 1)
+		(exclude_from_sim no)
+		(in_bom yes)
+		(on_board yes)
+		(dnp no)
+		(fields_autoplaced yes)
+		(property "Reference" "#PWR036"
+			(at 214.63 60.96 0)
+			(effects
+				(font
+					(size 1.27 1.27)
+				)
+				(hide yes)
+			)
+		)
+		(property "Value" "+1V8"
+			(at 214.63 52.07 0)
+			(effects
+				(font
+					(size 1.27 1.27)
+				)
+			)
+		)
+		(property "Footprint" ""
+			(at 214.63 57.15 0)
+			(effects
+				(font
+					(size 1.27 1.27)
+				)
+				(hide yes)
+			)
+		)
+		(property "Datasheet" ""
+			(at 214.63 57.15 0)
+			(effects
+				(font
+					(size 1.27 1.27)
+				)
+				(hide yes)
+			)
+		)
+		(property "Description" "Power symbol creates a global label with name \"+1V8\""
+			(at 214.63 57.15 0)
+			(effects
+				(font
+					(size 1.27 1.27)
+				)
+				(hide yes)
+			)
+		)
+		(pin "1"
+		)
+		(instances
+			(project "Digitiyer_demo_1V8_module"
+				(path "/9366839b-90ab-4146-a727-74c5e521354c"
+					(reference "#PWR036")
+					(unit 1)
+				)
+			)
+		)
+	)
+	(symbol
 		(lib_id "power:GND")
 		(at 179.07 115.57 0)
@@
 			)
 		)
-		(property "Footprint" "Package_TO_SOT_SMD:SOT-23-3"
+		(property "Footprint" "Package_TO_SOT_SMD:SOT-323_SC-70_Handsoldering"
 			(at 196.85 114.3 0)
 			(effects

Commit message: uklad
Parts:
- added C39: 10uF, Capacitor_SMD:C_0402_1005Metric, symbol Device:C_Small
- added C40: 100nF, Capacitor_SMD:C_0603_1608Metric, symbol Device:C_Small
- added D8: LED_Small, symbol Device:LED_Small
- R20: footprint Capacitor_SMD:C_0603_1608Metric -> Resistor_SMD:R_0603_1608Metric
- R27, R9: footprint Capacitor_SMD:C_0402_1005Metric -> Resistor_SMD:R_0402_1005Metric
Connections:
- net +1V8: now also C39.2, C40.1
- net GND: now also C39.1, C40.2, D8.1 (K)
- net at U4.14 (P03): now also D8.2 (A)
- no-connect marks 30 -> 29
Other:
- note added: "PPD"

Commit message: finální uložení?
Parts:
- D8: footprint (none) -> LED_SMD:LED_0603_1608Metric
- FB1, FB2, FB3: footprint Capacitor_SMD:C_0805_2012Metric -> Inductor_SMD:L_0805_2012Metric

Commit message: save
Parts:
- C31, C33: footprint Capacitor_SMD:C_0603_1608Metric -> Capacitor_SMD:C_0805_2012Metric
Changed lines of the file:
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@@
 			)
 		)
-		(property "Footprint" "Capacitor_SMD:C_0603_1608Metric"
+		(property "Footprint" "Capacitor_SMD:C_0805_2012Metric"
 			(at 199.39 95.25 0)
 			(effects
@@
 			)
 		)
-		(property "Footprint" "Capacitor_SMD:C_0603_1608Metric"
+		(property "Footprint" "Capacitor_SMD:C_0805_2012Metric"
 			(at 179.07 110.49 0)
 			(effects
